File: controlbox/vfd/vfdinterface/vfdinterface.kicad_pcb (KiCad board)
At the start: 0 parts

Commit message: Place components.
Parts:
- added C1: 100n, Capacitor_SMD_AKL:C_0603_1608Metric, F.Cu at (65.8, 73.2)
- added C2: 100n, Capacitor_SMD_AKL:C_0603_1608Metric, F.Cu at (55.3, 73.3)
- added D1: 1N4148, Diode_SMD_AKL:D_MiniMELF, F.Cu at (65.9, 55.8)
- added H1: MountingHole, MountingHole:MountingHole_3.2mm_M3, F.Cu at (79.6, 71.7)
- added J1: Conn_01x04, Connector_JST:JST_XH_B4B-XH-A_1x04_P2.50mm_Vertical, F.Cu at (80.4, 56.2)
- added J2: Conn_01x03, Connector_JST:JST_XH_B3B-XH-A_1x03_P2.50mm_Vertical, F.Cu at (67.9, 67.4)
- added J3: Conn_01x02, Connector_JST:JST_XH_B2B-XH-A_1x02_P2.50mm_Vertical, F.Cu at (70.5, 56.0)
- added Q2: BSS138, Package_TO_SOT_SMD_AKL:SOT-23, F.Cu at (66.6, 62.2)
- added R1: 10K, Resistor_SMD_AKL:R_0603_1608Metric, F.Cu at (70.3, 61.2)
- added R2: 1K, Resistor_SMD_AKL:R_0603_1608Metric, F.Cu at (70.3, 63.1)
- added R3: 100k, Resistor_SMD_AKL:R_0603_1608Metric, F.Cu at (70.2, 72.4)
- added RLY1: Siemens V23101-A0006-B101, w_relay:relay_V23101-D0-B, F.Cu at (59.0, 60.9)
- added U1: TLC271ACP, Package_SO_AKL:SO-8_3.9x4.9mm_P1.27mm, F.Cu at (60.4, 72.1)
Other:
- board outline added: 29.7 x 22.7 mm
- copper layers 0 -> 2
