File: controlbox/vfd/vfdinterface/vfdinterface.kicad_sch (KiCad schematic)
At the start: 12 parts, among them J1 Conn_01x04, J2 Conn_01x03, J3 Conn_01x02, Q2 BSS138, U1 TLC271ACP

Commit message: Place components.
Parts:
- added H1: MountingHole, MountingHole:MountingHole_3.2mm_M3, symbol Mechanical:MountingHole
- RLY1: footprint (none) -> w_relay:relay_V23101-D0-B; symbol w_relay:RELAY_V23101-D0 -> w_relay:RELAY_V23101-D0-B
- U1: footprint Package_DIP_AKL:DIP-8_W7.62mm_LongPads -> Package_SO_AKL:SO-8_3.9x4.9mm_P1.27mm; symbol Amplifier_Operational_AKL:TLC271ACP -> Amplifier_Operational_AKL:TLC271ACD
Connections:
- net at D1.2 (A), Q2.3 (D): now also RLY1.12; no longer RLY1.2
- net at J1.2 (Pin_2): now also RLY1.2; no longer RLY1.12
Changed lines of the file:
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@@
 	)
 	(symbol
-		(lib_id "Amplifier_Operational_AKL:TLC271ACP")
+		(lib_id "Amplifier_Operational_AKL:TLC271ACD")
 		(at 124.46 127 0)
 		(unit 1)
@@
 			)
 		)
-		(property "Footprint" "Package_DIP_AKL:DIP-8_W7.62mm_LongPads"
+		(property "Footprint" "Package_SO_AKL:SO-8_3.9x4.9mm_P1.27mm"
 			(at 124.46 127 0)
 			(effects
@@
 			)
 		)
-		(property "Description" "DIP-8 CMOS Low Power Operational Amplifier, Selectable Bias Current, 5mV Offset, 2.5MHz GBW, Alternate KiCAD Library"
+		(property "Description" "SO-8 CMOS Low Power Operational Amplifier, Selectable Bias Current, 5mV Offset, 2.5MHz GBW, Alternate KiCAD Library"
 			(at 124.46 127 0)
 			(effects
@@
 	)
 	(symbol
-		(lib_id "w_relay:RELAY_V23101-D0")
+		(lib_id "w_relay:RELAY_V23101-D0-B")
 		(at 135.89 63.5 270)
 		(mirror x)
@@
 			)
 		)
-		(property "Footprint" ""
+		(property "Footprint" "w_relay:relay_V23101-D0-B"
 			(at 135.89 63.5 0)
 			(effects
@@
 			)
 		)
-		(property "Description" "V23101-D0 relay"
+		(property "Description" "1 Form B relay, TE V23101-D0-xB"
 			(at 135.89 63.5 0)
 			(effects
@@
 					(unit 1)
 				)
+			)
+		)
+	)
+	(symbol
+		(lib_id "Mechanical:MountingHole")
+		(at 86.614 96.774 0)
+		(unit 1)
+		(exclude_from_sim no)
+		(in_bom yes)
+		(on_board yes)
+		(dnp no)
+		(fields_autoplaced yes)
+		(property "Reference" "H1"
+			(at 90.17 95.5039 0)
+			(effects
+				(font
+					(size 1.27 1.27)
+				)
+				(justify left)
+			)
+		)
+		(property "Value" "MountingHole"
+			(at 90.17 98.0439 0)
+			(effects
+				(font
+					(size 1.27 1.27)
+				)
+				(justify left)
+			)
+		)
+		(property "Footprint" "MountingHole:MountingHole_3.2mm_M3"
+			(at 86.614 96.774 0)
+			(effects
+				(font
+					(size 1.27 1.27)
+				)
+				(hide yes)
+			)
+		)
+		(property "Datasheet" "~"
+			(at 86.614 96.774 0)
+			(effects
+				(font
+					(size 1.27 1.27)
+				)
+				(hide yes)
+			)
+		)
+		(property "Description" "Mounting Hole without connection"
+			(at 86.614 96.774 0)
+			(effects
+				(font
+					(size 1.27 1.27)
+				)
+				(hide yes)
+			)
+		)
+		(instances
+			(project "vfdinterface"
+				(path "/b81aded0-bd17-4345-984b-f1ee8de72aca"
+					(reference "H1")
+					(unit 1)
+				)

Commit message: Finish routing.
Parts:
- renumbered Q2 to Q1
Changed lines of the file:
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@@
 		(dnp no)
 		(fields_autoplaced yes)
-		(property "Reference" "Q2"
+		(property "Reference" "Q1"
 			(at 136.525 77.4699 0)
 			(effects
@@
 			(project "vfdinterface"
 				(path "/b81aded0-bd17-4345-984b-f1ee8de72aca"
-					(reference "Q2")
+					(reference "Q1")
 					(unit 1)
 				)

Commit message: Fix opamp gain.
Parts:
- added R4: 51k, Resistor_SMD_AKL:R_0603_1608Metric, symbol Resistor_AKL:R_0603
- added R5: 22k, Resistor_SMD_AKL:R_0603_1608Metric, symbol Resistor_AKL:R_0603
Connections:
- net GND: now also R5.1
- net at J1.3 (Pin_3), U1.6: now also R4.2; no longer U1.2 (-)
- new net: R4.1, R5.2, U1.2 (-)
Changed lines of the file:
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@@
 	(version 20231120)
 	(generator "eeschema")
-	(generator_version "7.99")
+	(generator_version "8.99")
 	(paper "A4")
 	(junction
@@
 	)
 	(junction
+		(at 116.84 111.76)
+		(diameter 0)
+		(color 0 0 0 0)
+	)
+	(junction
 		(at 88.9 66.04)
 		(diameter 0)
@@
 	(wire
 		(pts
-			(xy 116.84 111.76) (xy 134.62 111.76)
-		)
-		(stroke
-			(width 0)
-			(type default)
-		)
-	)
-	(wire
-		(pts
 			(xy 124.46 53.34) (xy 132.08 53.34)
 		)
@@
 	(wire
 		(pts
+			(xy 129.54 111.76) (xy 134.62 111.76)
+		)
+		(stroke
+			(width 0)
+			(type default)
+		)
+	)
+	(wire
+		(pts
+			(xy 101.6 114.3) (xy 101.6 111.76)
+		)
+		(stroke
+			(width 0)
+			(type default)
+		)
+	)
+	(wire
+		(pts
 			(xy 149.86 49.53) (xy 149.86 53.34)
 		)
@@
 	(wire
 		(pts
+			(xy 116.84 111.76) (xy 121.92 111.76)
+		)
+		(stroke
+			(width 0)
+			(type default)
+		)
+	)
+	(wire
+		(pts
 			(xy 121.92 134.62) (xy 121.92 139.7)
 		)
@@
 	(wire
 		(pts
+			(xy 111.76 111.76) (xy 116.84 111.76)
+		)
+		(stroke
+			(width 0)
+			(type default)
+		)
+	)
+	(wire
+		(pts
 			(xy 101.6 66.04) (xy 96.52 66.04)
 		)
@@
 		(pts
 			(xy 96.52 66.04) (xy 88.9 66.04)
+		)
+		(stroke
+			(width 0)
+			(type default)
+		)
+	)
+	(wire
+		(pts
+			(xy 101.6 111.76) (xy 104.14 111.76)
 		)
 		(stroke
@@
 	(symbol
 		(lib_id "Resistor_AKL:R_0603")
+		(at 107.95 111.76 90)
+		(unit 1)
+		(exclude_from_sim no)
+		(in_bom yes)
+		(on_board yes)
+		(dnp no)
+		(property "Reference" "R5"
+			(at 106.426 109.22 90)
+			(effects
+				(font
+					(size 1.27 1.27)
+				)
+			)
+		)
+		(property "Value" "22k"
+			(at 107.696 111.76 90)
+			(effects
+				(font
+					(size 1.27 1.27)
+				)
+			)
+		)
+		(property "Footprint" "Resistor_SMD_AKL:R_0603_1608Metric"
+			(at 119.38 111.76 0)
+			(effects
+				(font
+					(size 1.27 1.27)
+				)
+				(hide yes)
+			)
+		)
+		(property "Datasheet" "~"
+			(at 107.95 111.76 0)
+			(effects
+				(font
+					(size 1.27 1.27)
+				)
+				(hide yes)
+			)
+		)
+		(property "Description" "SMD 0603 Chip Resistor, European Symbol, Alternate KiCad Library"
+			(at 107.95 111.76 0)
+			(effects
+				(font
+					(size 1.27 1.27)
+				)
+				(hide yes)
+			)
+		)
+		(pin "2"
+		)
+		(pin "1"
+		)
+		(instances
+			(project "vfdinterface"
+				(path "/b81aded0-bd17-4345-984b-f1ee8de72aca"
+					(reference "R5")
+					(unit 1)
+				)
+			)
+		)
+	)
+	(symbol
+		(lib_id "Resistor_AKL:R_0603")
 		(at 102.87 129.54 90)
 		(unit 1)
@@
 		(on_board yes)
 		(dnp no)
-		(fields_autoplaced yes)
 		(property "Reference" "R3"
-			(at 102.87 123.19 90)
+			(at 101.346 127.254 90)
 			(effects
 				(font
@@
 		)
 		(property "Value" "100k"
-			(at 102.87 125.73 90)
+			(at 102.87 129.54 90)
 			(effects
 				(font
@@
 					(unit 1)
 				)
+			)
+		)
+	)
+	(symbol
+		(lib_id "Resistor_AKL:R_0603")
+		(at 125.73 111.76 90)
+		(unit 1)
+		(exclude_from_sim no)
+		(in_bom yes)
+		(on_board yes)
+		(dnp no)
+		(property "Reference" "R4"
+			(at 124.206 109.474 90)
+			(effects
+				(font
+					(size 1.27 1.27)
+				)
+			)
+		)
+		(property "Value" "51k"
+			(at 125.73 111.76 90)
+			(effects
+				(font
+					(size 1.27 1.27)
+				)
+			)
+		)
+		(property "Footprint" "Resistor_SMD_AKL:R_0603_1608Metric"
+			(at 137.16 111.76 0)
+			(effects
+				(font
+					(size 1.27 1.27)
+				)
+				(hide yes)
+			)
+		)
+		(property "Datasheet" "~"
+			(at 125.73 111.76 0)
+			(effects
+				(font
+					(size 1.27 1.27)
+				)
+				(hide yes)
+			)
+		)
+		(property "Description" "SMD 0603 Chip Resistor, European Symbol, Alternate KiCad Library"
+			(at 125.73 111.76 0)
+			(effects
+				(font
+					(size 1.27 1.27)
+				)
+				(hide yes)
+			)
+		)
+		(pin "2"
+		)
+		(pin "1"
+		)
+		(instances
+			(project "vfdinterface"
+				(path "/b81aded0-bd17-4345-984b-f1ee8de72aca"
+					(reference "R4")
+					(unit 1)
+				)
+			)
+		)
+	)
+	(symbol
+		(lib_id "power:GND")
+		(at 101.6 114.3 0)
+		(unit 1)
+		(exclude_from_sim no)
+		(in_bom yes)
+		(on_board yes)
+		(dnp no)
+		(fields_autoplaced yes)
+		(property "Reference" "#PWR07"
+			(at 101.6 120.65 0)
+			(effects
+				(font
+					(size 1.27 1.27)
+				)
+				(hide yes)
+			)
+		)
+		(property "Value" "GND"
+			(at 101.6 119.38 0)
+			(effects
+				(font
+					(size 1.27 1.27)
+				)
+			)
+		)
+		(property "Footprint" ""
+			(at 101.6 114.3 0)
+			(effects
+				(font
+					(size 1.27 1.27)
+				)
+				(hide yes)
+			)
+		)
+		(property "Datasheet" ""
+			(at 101.6 114.3 0)
+			(effects
+				(font
+					(size 1.27 1.27)
+				)
+				(hide yes)
+			)
+		)
+		(property "Description" "Power symbol creates a global label with name \"GND\" , ground"
+			(at 101.6 114.3 0)
+			(effects
+				(font
+					(size 1.27 1.27)
+				)
+				(hide yes)
+			)
+		)
+		(pin "1"
+		)
+		(instances
+			(project "vfdinterface"
+				(path "/b81aded0-bd17-4345-984b-f1ee8de72aca"
+					(reference "#PWR07")
+					(unit 1)
+				)

Commit message: Change to DIL package.
Parts:
- U1: footprint Package_SO_AKL:SO-8_3.9x4.9mm_P1.27mm -> Package_DIP_AKL:DIP-8_W7.62mm
Changed lines of the file:
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@@
 			)
 		)
-		(property "Footprint" "Package_SO_AKL:SO-8_3.9x4.9mm_P1.27mm"
+		(property "Footprint" "Package_DIP_AKL:DIP-8_W7.62mm"
 			(at 124.46 127 0)
 			(effects
